File: fiero-wiper-pulse-board.kicad_sch (KiCad schematic)
At the start: 0 parts

Commit message: Add schematic and project settings for wiper pulse board
Added initial KiCad schematic with resistors, connectors, and GND symbols for the Fiero wiper pulse board. Project settings were updated to include ERC rules, BOM export configuration, and sheet metadata. A backup of the project was also created.
Parts:
- added J1: Conn_01x04_Pin, symbol Connector:Conn_01x04_Pin
- added J2: Conn_01x04_Socket, symbol Connector:Conn_01x04_Socket
- added J3: Conn_01x01_Socket, symbol Connector:Conn_01x01_Socket
- added R1, R6: 33k, symbol Device:R_US
- added R2: 15k, symbol Device:R_US
- added R9: 560, symbol Device:R_US
Connections:
- new net: J1.4 (Pin_4), J2.4 (Pin_4), R9.1
- new net: J1.1 (Pin_1), R6.1
- new net: J1.2 (Pin_2), J2.2 (Pin_2)
- new net GND: J3.1 (Pin_1), R9.2
